Commit message: updated robot model : ears and some joint position

File: src/assignment2/urdf/robotDog.xacro (robot description, xacro)
@@ -9,4 +9,36 @@
                 iyy="${mass*(3*r*r+l*l)/12}" iyz = "0" izz="${mass*(r*r)/2}" />
  </xacro:macro>
+ <xacro:macro name="link_ear" params="name">
+   <link name="${name}">
+            <inertial>
+              <mass value="0.2"/>
+              <origin rpy="0 0 0" xyz="0 0 0"/>
+              <inertia ixx="0.000526666666667" ixy="0" ixz="0" iyy="0.000526666666667" iyz="0" izz="0.001"/>
+            </inertial>
+            <collision name="${name}_collision">
+              <origin rpy="0 0 1.5708" xyz="0 0 0"/>
+              <geometry>
+                <box size="0.034 0.05 0.03"/>
+              </geometry>
+            </collision>
+            <visual name="${name}_visual">
+              <origin rpy="0 0 0" xyz="0 0 0"/>
+              <geometry>
+                <box size="0.034 0.05 0.03"/>
+              </geometry>
+		<material name="blue" />
+            </visual>
+        </link>
+ </xacro:macro>
+    <xacro:macro name="joint_ear" params="name child origin_xyz">
+      <joint name="${name}" type="fixed">
+        <origin rpy="0 0 0" xyz="${origin_xyz}"/>
+        <child link="${child}"/>
+        <parent link="head_link"/>
+        <axis rpy="0 0 0" xyz="0 0 1"/>
+        <limit effort="10000" velocity="1000"/>
+        <joint_properties damping="1.0" friction="1.0"/>
+      </joint>
+    </xacro:macro>
     <xacro:macro name="link_wheel" params="name">
         <link name="${name}">
@@ -40,4 +72,5 @@
       </joint>
     </xacro:macro>
+<!-- base link  -->
   <link name="base_link">
     <!-- pose and inertial -->
@@ -113,5 +146,5 @@
   	<axis xyz="0 0 1"/>
   	<limit effort="1000.0" lower="-3.14" upper="3.14" velocity="0.2"/>
-  	<origin rpy="0 0 0" xyz="0 0 0.035"/> <!-- half the height of the base link -->
+  	<origin rpy="0 0 0" xyz="0.15 0 0.035"/> <!-- half the height of the base link -->
   	<parent link="base_link"/>
   	<child link="neck_link"/>
@@ -125,5 +158,5 @@
   	</inertial>
   	<collision>
-  	  <origin xyz="0 0 0.04" rpy="0 0 1.57"/> <!-- frame moved to the base of the head -->
+  	  <origin xyz="0 0 0.04" rpy="0 0 0"/> <!-- frame moved to the base of the head -->
       <geometry>
         <box size="0.034 0.2 0.08"/>
@@ -131,5 +164,5 @@
   	</collision>
   	<visual>
-  	  <origin xyz="0 0 0.04" rpy="0 0 1.57"/> <!-- frame moved to the base of the head -->
+  	  <origin xyz="0 0 0.04" rpy="0 0 0"/> <!-- frame moved to the base of the head -->
       <geometry>
         <box size="0.034 0.2 0.08"/>
@@ -168,8 +201,13 @@
   <joint name="camera_joint" type="fixed">
     <axis xyz="0 1 0" />
-    <origin xyz="0 0.017 0.04" rpy="0 0 1.5708"/>
+    <origin xyz="0 0.017 0.04" rpy="0 0 0"/>
     <parent link="head_link"/>
     <child link="camera_link"/>
   </joint>
+<!-- hears definition -->
+  <xacro:link_ear name="link_right_ear" />
+  <xacro:link_ear name="link_left_ear" />
+  <xacro:joint_ear name="joint_right_ear"  child="link_right_ear"  origin_xyz="0 0.08 0.08"  />
+  <xacro:joint_ear name="joint_left_ear"   child="link_left_ear"   origin_xyz="0 -0.08 0.08"  />
 <!-- transmission -->
 <transmission name="head_joint_trans">

Commit message: finished the robot model description and started to implement a navigation action server, which is gonna substitute the old navigation service

File: src/assignment2/urdf/robotDog.xacro (robot description, xacro)
@@ -3,16 +3,24 @@
  <xacro:include filename="$(find assignment2)/urdf/materials.xacro" />
  <xacro:include filename="$(find assignment2)/urdf/robotDog.gazebo" />
+ <xacro:property name="length_wheel" value="0.04" />
+ <xacro:property name="radius_wheel" value="0.1" />
+ <xacro:property name="neck_length" value="0.15" />
+ <xacro:property name="neck_radius" value="0.05" />
  <xacro:property name="camera_link" value="0.05" /> <!-- Size of square 'camera' box -->
- <xacro:property name="neck_length" value="0.15" />
  <xacro:macro name="cylinder_inertia" params="mass r l">
     <inertia ixx="${mass*(3*r*r+l*l)/12}" ixy = "0" ixz = "0"
                 iyy="${mass*(3*r*r+l*l)/12}" iyz = "0" izz="${mass*(r*r)/2}" />
  </xacro:macro>
+ <xacro:macro name="box_inertia" params="mass w h d">
+    <inertia ixx="${mass*(h*h+d*d)/12}" ixy = "0" ixz = "0"
+                iyy="${mass*(w*w+d*d)/12}" iyz = "0" izz="${mass*(w*w+h*h)/12}" />
+ </xacro:macro>
  <xacro:macro name="link_ear" params="name">
    <link name="${name}">
             <inertial>
-              <mass value="0.2"/>
+              <mass value="0.1"/>
               <origin rpy="0 0 0" xyz="0 0 0"/>
-              <inertia ixx="0.000526666666667" ixy="0" ixz="0" iyy="0.000526666666667" iyz="0" izz="0.001"/>
+              <!-- <inertia ixx="0.000526666666667" ixy="0" ixz="0" iyy="0.000526666666667" iyz="0" izz="0.001"/> -->
+	      <xacro:box_inertia mass="0.1" w="0.05" h="0.03" d="0.034"/>
             </inertial>
             <collision name="${name}_collision">
@@ -46,10 +54,11 @@
               <mass value="0.2"/>
               <origin rpy="0 1.5707 1.5707" xyz="0 0 0"/>
-              <inertia ixx="0.000526666666667" ixy="0" ixz="0" iyy="0.000526666666667" iyz="0" izz="0.001"/>
+              <!-- <inertia ixx="0.000526666666667" ixy="0" ixz="0" iyy="0.000526666666667" iyz="0" izz="0.001"/> -->
+	      <xacro:cylinder_inertia mass="0.2" r="${radius_wheel}" l="${length_wheel}" />
             </inertial>
             <collision name="link_right_wheel_collision">
               <origin rpy="0 1.5707 1.5707" xyz="0 0 0"/>
               <geometry>
-                <cylinder length="0.04" radius="0.1"/>
+                <cylinder length="${length_wheel}" radius="${radius_wheel}"/>
               </geometry>
             </collision>
@@ -57,5 +66,5 @@
               <origin rpy="0 1.5707 1.5707" xyz="0 0 0"/>
               <geometry>
-                <cylinder length="0.04" radius="0.1"/>
+                <cylinder length="${length_wheel}" radius="${radius_wheel}"/>
               </geometry>
             </visual>
@@ -72,5 +81,5 @@
       </joint>
     </xacro:macro>
-<!-- base link  -->
+<!-- _______________base link____________________  -->
   <link name="base_link">
     <!-- pose and inertial -->
@@ -122,21 +131,22 @@
   <xacro:joint_wheel name="joint_right_wheel"  child="link_right_wheel"  origin_xyz="-0.05 0.15 0"  />
   <xacro:joint_wheel name="joint_left_wheel"   child="link_left_wheel"   origin_xyz="-0.05 -0.15 0"  />
-<!--neck definition -->
+<!-- _______________neck definition_______________ -->
   <link name="neck_link">
   	<inertial>
   		<mass value="0.025"/>
   		<origin xyz="0 0 0" rpy="0 0 0" />
-  		<inertia ixx="0.000010279" ixy="0" ixz="0" iyy="0.000010279" iyz="0" izz="0.000007225"/>
+  		<!--<inertia ixx="0.000010279" ixy="0" ixz="0" iyy="0.000010279" iyz="0" izz="0.000007225"/>-->
+		<xacro:cylinder_inertia mass="0.2" r="${neck_radius}" l="${neck_length}" />
   	</inertial>
   	<collision>
-  	  <origin xyz="0 0 0.075" rpy="0 0 0"/> <!-- frame moved to the base of the cylinder -->
-      <geometry>
-        <cylinder radius="0.04" length="${neck_length}"/>
+  	  <origin xyz="0 0 ${neck_length/2}" rpy="0 0 0"/> <!-- frame moved to the base of the cylinder -->
+      <geometry>
+        <cylinder radius="${neck_radius}" length="${neck_length}"/>
       </geometry>
   	</collision>
   	<visual>
-  	  <origin xyz="0 0 0.075" rpy="0 0 0"/> <!-- frame moved to the base of the cylinder -->
-      <geometry>
-        <cylinder radius="0.04" length="${neck_length}"/>
+  	  <origin xyz="0 0 ${neck_length/2}" rpy="0 0 0"/> <!-- frame moved to the base of the cylinder -->
+      <geometry>
+        <cylinder radius="${neck_radius}" length="${neck_length}"/>
       </geometry>
       <material name="red" />
@@ -155,5 +165,5 @@
   		<mass value="0.025"/>
   		<origin xyz="0 0 0" rpy="0 0 0" />
-  		<inertia ixx="0.000010279" ixy="0" ixz="0" iyy="0.000010279" iyz="0" izz="0.000007225"/>
+  		<xacro:box_inertia mass="0.025" w="0.2" h="0.08" d="0.034"/>
   	</inertial>
   	<collision>

Commit message: fixed error during switch from NORMAL to PLAY state and the problem regurding the head montions

File: src/assignment2/urdf/robotDog.xacro (robot description, xacro)
@@ -163,5 +163,5 @@
     <link name="head_link">
   	<inertial>
-  		<mass value="0.025"/>
+  		<mass value="0.0025"/>
   		<origin xyz="0 0 0" rpy="0 0 0" />
   		<xacro:box_inertia mass="0.025" w="0.2" h="0.08" d="0.034"/>
@@ -211,13 +211,15 @@
   <joint name="camera_joint" type="fixed">
     <axis xyz="0 1 0" />
-    <origin xyz="0 0.017 0.04" rpy="0 0 0"/>
+    <origin xyz="0.017 0 0.04" rpy="0 0 0"/>
     <parent link="head_link"/>
     <child link="camera_link"/>
   </joint>
 <!-- hears definition -->
+<!--
   <xacro:link_ear name="link_right_ear" />
   <xacro:link_ear name="link_left_ear" />
   <xacro:joint_ear name="joint_right_ear"  child="link_right_ear"  origin_xyz="0 0.08 0.08"  />
   <xacro:joint_ear name="joint_left_ear"   child="link_left_ear"   origin_xyz="0 -0.08 0.08"  />
+-->
 <!-- transmission -->
 <transmission name="head_joint_trans">

Commit message: Fixed the switch from Normal to Play states

File: src/assignment2/urdf/robotDog.xacro (robot description, xacro)
@@ -163,5 +163,5 @@
     <link name="head_link">
   	<inertial>
-  		<mass value="0.0025"/>
+  		<mass value="0.025"/>
   		<origin xyz="0 0 0" rpy="0 0 0" />
   		<xacro:box_inertia mass="0.025" w="0.2" h="0.08" d="0.034"/>

Commit message: final commit

File: src/assignment2/urdf/robotDog.xacro (robot description, xacro)
@@ -3,4 +3,8 @@
  <xacro:include filename="$(find assignment2)/urdf/materials.xacro" />
  <xacro:include filename="$(find assignment2)/urdf/robotDog.gazebo" />
+ <xacro:property name="chassis_length" value="0.5" />
+ <xacro:property name="chassis_width" value="0.3" />
+ <xacro:property name="chassis_height" value="0.07" />
+ <xacro:property name="chassis_mass" value="6" />
  <xacro:property name="length_wheel" value="0.04" />
  <xacro:property name="radius_wheel" value="0.1" />
@@ -88,9 +92,10 @@
       <mass value="5"/>
       <origin rpy="0 0 0" xyz="0 0 0.1"/>
-      <inertia ixx="0.0395416666667" ixy="0" ixz="0" iyy="0.106208333333" iyz="0" izz="0.106208333333"/>
+      <!--<inertia ixx="0.0395416666667" ixy="0" ixz="0" iyy="0.106208333333" iyz="0" izz="0.106208333333"/> -->
+      <xacro:box_inertia mass="${chassis_mass}" w="${chassis_length}" h="${chassis_width}" d="${chassis_height}"/>
     </inertial>
     <collision name="collision_chassis">
       <geometry>
-        <box size="0.5 0.3 0.07"/>
+        <box size="${chassis_length} ${chassis_width} ${chassis_height}"/>
       </geometry>
     </collision>
@@ -98,5 +103,5 @@
       <origin rpy="0 0 0" xyz="0 0 0"/>
       <geometry>
-        <box size="0.5 0.3 0.07"/>
+        <box size="${chassis_length} ${chassis_width} ${chassis_height}"/>
       </geometry>
       <material name="blue"/>
@@ -134,5 +139,5 @@
   <link name="neck_link">
   	<inertial>
-  		<mass value="0.025"/>
+  		<mass value="0.3"/>
   		<origin xyz="0 0 0" rpy="0 0 0" />
   		<!--<inertia ixx="0.000010279" ixy="0" ixz="0" iyy="0.000010279" iyz="0" izz="0.000007225"/>-->
@@ -163,7 +168,7 @@
     <link name="head_link">
   	<inertial>
-  		<mass value="0.025"/>
+  		<mass value="0.1"/>
   		<origin xyz="0 0 0" rpy="0 0 0" />
-  		<xacro:box_inertia mass="0.025" w="0.2" h="0.08" d="0.034"/>
+  		<xacro:box_inertia mass="0.1" w="0.2" h="0.08" d="0.034"/>
   	</inertial>
   	<collision>
