Commit message: tuned the move base params but sometimes the algo requires too much time to recognize that the robot is arrived in the goal position

File: src/final_assignment/urdf/robotDog.xacro (robot description, xacro)
@@ -79,5 +79,5 @@
         <origin rpy="0 0 0" xyz="${origin_xyz}"/>
         <child link="${child}"/>
-        <parent link="base_link"/>
+        <parent link="link_chassis"/>
         <axis rpy="0 0 0" xyz="0 1 0"/>
         <limit effort="10000" velocity="1000"/>
@@ -86,5 +86,5 @@
     </xacro:macro>
 <!-- _______________base link____________________  -->
-  <link name="base_link">
+  <link name="link_chassis">
     <!-- pose and inertial -->
     <pose>0 0 0.1 0 0 0</pose>
@@ -162,5 +162,5 @@
   	<limit effort="1000.0" lower="-3.14" upper="3.14" velocity="0.2"/>
   	<origin rpy="0 0 0" xyz="0.15 0 0.035"/> <!-- half the height of the base link -->
-  	<parent link="base_link"/>
+  	<parent link="link_chassis"/>
   	<child link="neck_link"/>
   </joint>
@@ -262,5 +262,5 @@
 	    <axis xyz="0 1 0" />
 	    <origin xyz="0.27 0 0.025" rpy="0 0 0"/>
-	    <parent link="base_link"/>
+	    <parent link="link_chassis"/>
 	    <child link="hokuyo_link"/>
 	 </joint>
